File: XMOS_demo/mcu.kicad_sch (KiCad schematic)
At the start: 47 parts, among them J1 XSYS2 DEBUG CONNECTOR, U1 U316-1024-QF60B, U2 W25Q32JVSS, Y1 Crystal_24M

Commit message: finished sch, pcb work
Parts:
- removed R4, R6: 0R, Resistor_SMD:R_0603_1608Metric, symbol Device:R_Small
- C1, C14, C15, C16: footprint Capacitor_SMD:C_0603_1608Metric -> Capacitor_SMD:C_0402_1005Metric
- C10: renamed from C11; footprint Capacitor_SMD:C_0603_1608Metric -> Capacitor_SMD:C_0402_1005Metric
- C11: renamed from C12; footprint Capacitor_SMD:C_0603_1608Metric -> Capacitor_SMD:C_0402_1005Metric
- C12: renamed from C13; footprint Capacitor_SMD:C_0603_1608Metric -> Capacitor_SMD:C_0402_1005Metric
- C13: renamed from C2; footprint Capacitor_SMD:C_0603_1608Metric -> Capacitor_SMD:C_0402_1005Metric
- C2: renamed from C3; footprint Capacitor_SMD:C_0603_1608Metric -> Capacitor_SMD:C_0402_1005Metric
- C3: renamed from C4; footprint Capacitor_SMD:C_0603_1608Metric -> Capacitor_SMD:C_0402_1005Metric
- C4: renamed from C5; footprint Capacitor_SMD:C_0603_1608Metric -> Capacitor_SMD:C_0402_1005Metric
- C5: renamed from C6; footprint Capacitor_SMD:C_0603_1608Metric -> Capacitor_SMD:C_0402_1005Metric
- C6: renamed from C7; footprint Capacitor_SMD:C_0603_1608Metric -> Capacitor_SMD:C_0402_1005Metric
- C7: renamed from C8; footprint Capacitor_SMD:C_0603_1608Metric -> Capacitor_SMD:C_0402_1005Metric
- C8: renamed from C9; footprint Capacitor_SMD:C_0603_1608Metric -> Capacitor_SMD:C_0402_1005Metric
- C9: renamed from C10; footprint Capacitor_SMD:C_0603_1608Metric -> Capacitor_SMD:C_0402_1005Metric
- U1: footprint _QFN:QFN-60_7x7mm_P0.4mm_EP_ThermalVias_PowerBars -> _Package_QFN:QFN-60_7x7mm_P0.4mm_EP_ThermalVias_PowerBars
- renumbered R12 to R10, R13 to R11, R14 to R12, R15 to R13, R16 to R14, R17 to R15, R5 to R4, R7 to R5, R8 to R6, R9 to R7, R10 to R8, R11 to R9
Connections:
- net P_IO_L is gone; now on net P3V3: C1.2, C13.1, R4.2, U1.8 (VDDIOL), U2.8 (VCC)
- net I2S_LRCK: now reaches U1.10 (X1D01)
- net CODEC_~{RST}: now reaches U1.11 (X1D09)
- net I2S_SCLK: now reaches U1.13 (X1D10)
- net MCLK: now reaches U1.14 (X1D11)
- net I2S_ADC: now reaches U1.7 (X0D11)
- net I2S_DAC: now reaches U1.9 (X1D00)
- no-connect marks 1 -> 14
Other:
- note removed: "TAKE CARE WITH IO_L SUPPLY CONFIGURATION DEPENDING ON AVIABLE QSPI FLASH"
- moved on the sheet: C1, C10, C11, C12, C13, D1, D2, D3, FB1, R1, R2, R3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
