File: XMOS_demo/audio_out.kicad_sch (KiCad schematic)
At the start: 0 parts

Commit message: Work on audio output amplifier
Parts:
- added C27, C28, C29, C30, C31: 1u, Capacitor_SMD:C_0603_1608Metric, symbol Device:C_Small
- added C32: 100n, Capacitor_SMD:C_0603_1608Metric, symbol Device:C_Small
- added C33, C34, C35, C36: 470n, Capacitor_THT:C_Rect_L7.2mm_W8.5mm_P5.00mm_FKP2_FKP2_MKS2_MKP2, symbol Device:C_Small
- added R20, R21, R22, R23, R24: 0R, Resistor_SMD:R_0603_1608Metric, symbol Device:R_Small
- added RN1, RN2: 10k, Resistor_SMD:R_Array_Convex_4x1206, symbol Device:R_Pack04
- added U5: MAX97220C, Package_DFN_QFN:TQFN-16-1EP_3x3mm_P0.5mm_EP1.23x1.23mm_ThermalVias, symbol _Amplifier_Audio:MAX97220C
Connections:
- new net: C28.1, C29.1, C30.1, U5.1 (PVDD), U5.13 (SVDD), U5.9 (SVDD2)
- new net: C27.1, U5.2 (C1P)
- new net: C27.2, U5.4 (C1N)
- new net AMP_BIAS: C32.1, R20.2, U5.11 (BIAS)
- new net AMP_INL+: R23.2, RN2.2 (R2.1), RN2.3 (R3.1), U5.15 (INL+)
- new net AMP_INL-: R24.2, RN2.1 (R1.1), RN2.4 (R4.1), U5.14 (INL-)
- new net AMP_INR+: R21.2, RN1.2 (R2.1), RN1.3 (R3.1), U5.7 (INR+)
- new net AMP_INR-: R22.2, RN1.1 (R1.1), RN1.4 (R4.1), U5.8 (INR-)
- new net AMP_OUTL: RN2.8 (R1.2), U5.12 (OUTL)
- new net AMP_OUTR: RN1.8 (R1.2), U5.10 (OUTR)
- new net AMP_PVSS: C31.1, R20.1, U5.5 (PVSS)
- new net GND: C28.2, C29.2, C30.2, C31.2, C32.2, RN1.7 (R2.2), RN2.7 (R2.2), U5.17 (EPAD), U5.3 (PGND), U5.6 (SGND)
- new net INL+: C35.1
- new net INL-: C36.1
- new net INR+: C33.1
- new net INR-: C34.1
- new net R_INL+: C35.2, R23.1, RN2.6 (R3.2)
- new net R_INL-: C36.2, R24.1, RN2.5 (R4.2)
- new net R_INR+: C33.2, R21.1, RN1.6 (R3.2)
- new net R_INR-: C34.2, R22.1, RN1.5 (R4.2)
Other:
- note added: "REPLACE WITH 1u FOR MAX9722"
- note added: "TO USE WITH A/B/E VERSION OF MAX97220"

Commit message: Lots of sch work
Parts:
- added C38, C40, C41, C42: 470n, Capacitor_SMD:C_1206_3216Metric_Pad1.33x1.80mm_HandSolder, symbol Device:C_Small
- added J3: AudioJack3_SwitchT, _Connector_Audio:Jack_3.5mm_CUI_SJ-3523-SMT-TR_Horizontal, symbol Connector_Audio:AudioJack3_SwitchT
- added R26, R29: 0R, Resistor_SMD:R_0603_1608Metric, symbol Device:R_Small
- added R27: 10k, Resistor_SMD:R_0603_1608Metric, symbol Device:R_Small
- C32: Max Voltage 10V -> 16V
- U5: footprint Package_DFN_QFN:TQFN-16-1EP_3x3mm_P0.5mm_EP1.23x1.23mm_ThermalVias -> _QFN:TQFN-16-1EP_3x3mm_P0.5mm_EP1.23x1.23mm_ThermalVias
Connections:
- net AMP_OUTL: now also J3.T
- net AMP_OUTR: now also J3.R
- net GND: now also J3.S
- net INL+: now also C41.1
- net INL-: now also C42.1
- net INR+: now also C38.1
- net INR-: now also C40.1
- net R_INL+: now also C41.2
- net R_INL-: now also C42.2
- net R_INR+: now also C38.2
- net R_INR-: now also C40.2
- net P_AMP_SUPPLY: now reaches C28.1, C29.1, C30.1, U5.1 (PVDD), U5.13 (SVDD), U5.9 (SVDD2)
- net P_AMP_SUPPLY: now also R27.1, R29.1
- net at U5.16 (~{SHDN}): now also R26.2, R27.2
- new net P5V0: R29.2
- new net ~{SHDN}: R26.1
- no-connect marks 0 -> 1
Other:
- note added: "MOUNT EITHER FILM OR C0G CAPACITORS"
- note added: "MOUNT ONLY FOR MAX9722"
- moved on the sheet: C27, C28, C29, C30, C31, C32, C33, C34, C35, C36, R20, R21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

Commit message: sch work, pcb import and initial board outline
Changed lines of the file:
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@@
 		(dnp no)
 		(property "Reference" "R29"
-			(at 115.316 58.42 90)
+			(at 113.538 57.404 0)
 			(effects
 				(font
-					(size 1.016 1.016)
+					(size 1.27 1.27)
 				)
 			)
 		)
 		(property "Value" "0R"
-			(at 116.84 58.42 90)
+			(at 113.03 59.436 0)
 			(effects
 				(font
-					(size 0.762 0.762)
+					(size 1.27 1.27)
 				)
 			)

Commit message: sch mostly finished, needs tp, pcb component layout started
Parts:
- C31: renamed from C38; now fitted
- C35: renamed from C40; now fitted
- C36: renamed from C41; now fitted
- C37: renamed from C42; now fitted
- C38: renamed from C33; now not fitted
- C39: renamed from C34; now not fitted
- C40: renamed from C35; now not fitted
- C41: renamed from C36; now not fitted
- renumbered C28 to C32, C29 to C33, C30 to C34, C32 to C42, C27 to C43, C31 to C44, J3 to J4, R21 to R30, R22 to R31, R23 to R32, R24 to R33, R20 to R34, R27 to R35, R26 to R36, U5 to U7
Other:
- note added: "MOUNT EITHER FILM OR NP0 CAPACITORS"
- note removed: "MOUNT EITHER FILM OR C0G CAPACITORS"

Commit message: finished sch, pcb work
Parts:
- renumbered J4 to J5, R29 to R27, R30 to R28, R31 to R29, R32 to R30, R33 to R31, R34 to R32, R35 to R33, R36 to R34
Changed lines of the file:
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@@
 	)
 	(junction
+		(at 132.08 63.5)
+		(diameter 0)
+		(color 0 0 0 0)
+	)
+	(junction
 		(at 137.16 63.5)
 		(diameter 0)
@@
 	(wire
 		(pts
-			(xy 127 63.5) (xy 137.16 63.5)
+			(xy 127 63.5) (xy 132.08 63.5)
 		)
 		(stroke
@@
 	(wire
 		(pts
+			(xy 132.08 60.96) (xy 132.08 63.5)
+		)
+		(stroke
+			(width 0)
+			(type default)
+		)
+	)
+	(wire
+		(pts
 			(xy 106.68 116.84) (xy 114.3 116.84)
 		)
@@
 	(wire
 		(pts
+			(xy 132.08 63.5) (xy 137.16 63.5)
+		)
+		(stroke
+			(width 0)
+			(type default)
+		)
+	)
+	(wire
+		(pts
 			(xy 76.2 137.16) (xy 93.98 137.16)
 		)
@@
 		(on_board yes)
 		(dnp no)
-		(property "Reference" "#PWR061"
+		(property "Reference" "#PWR059"
 			(at 177.8 105.41 0)
 			(effects
@@
 			(project "XMOS_demo"
 				(path "/0a855fb0-ca19-4770-811e-70d8770d7fdd/82ce7187-f0cb-4a8a-9f6c-b1803f49d1ca"
-					(reference "#PWR061")
+					(reference "#PWR059")
 					(unit 1)
 				)
@@
 		(on_board yes)
 		(dnp no)
-		(property "Reference" "#PWR066"
+		(property "Reference" "#PWR064"
 			(at 93.98 166.37 0)
 			(effects
@@
 			(project "XMOS_demo"
 				(path "/0a855fb0-ca19-4770-811e-70d8770d7fdd/82ce7187-f0cb-4a8a-9f6c-b1803f49d1ca"
-					(reference "#PWR066")
+					(reference "#PWR064")
 					(unit 1)
 				)
@@
 		(on_board yes)
 		(dnp no)
-		(property "Reference" "R32"
+		(property "Reference" "R30"
 			(at 114.3 89.916 90)
 			(effects
@@
 			(project "XMOS_demo"
 				(path "/0a855fb0-ca19-4770-811e-70d8770d7fdd/82ce7187-f0cb-4a8a-9f6c-b1803f49d1ca"
-					(reference "R32")
+					(reference "R30")
 					(unit 1)
 				)
@@
 		(on_board yes)
 		(dnp no)
-		(property "Reference" "#PWR065"
+		(property "Reference" "#PWR063"
 			(at 93.98 143.51 0)
 			(effects
@@
 			(project "XMOS_demo"
 				(path "/0a855fb0-ca19-4770-811e-70d8770d7fdd/82ce7187-f0cb-4a8a-9f6c-b1803f49d1ca"
-					(reference "#PWR065")
+					(reference "#PWR063")
 					(unit 1)
 				)
@@
 		(on_board yes)
 		(dnp no)
-		(property "Reference" "R36"
+		(property "Reference" "R34"
 			(at 116.84 115.316 90)
 			(effects
@@
 			(project "XMOS_demo"
 				(path "/0a855fb0-ca19-4770-811e-70d8770d7fdd/82ce7187-f0cb-4a8a-9f6c-b1803f49d1ca"
-					(reference "R36")
+					(reference "R34")
 					(unit 1)
 				)
@@
 		(dnp no)
 		(fields_autoplaced yes)
-		(property "Reference" "#PWR058"
+		(property "Reference" "#PWR056"
 			(at 144.78 64.77 0)
 			(effects
@@
 			(project "XMOS_demo"
 				(path "/0a855fb0-ca19-4770-811e-70d8770d7fdd/82ce7187-f0cb-4a8a-9f6c-b1803f49d1ca"
-					(reference "#PWR058")
+					(reference "#PWR056")
 					(unit 1)
 				)
@@
 		(on_board yes)
 		(dnp no)
-		(property "Reference" "#PWR057"
+		(property "Reference" "#PWR055"
 			(at 116.84 57.15 0)
 			(effects
@@
 			(project "XMOS_demo"
 				(path "/0a855fb0-ca19-4770-811e-70d8770d7fdd/82ce7187-f0cb-4a8a-9f6c-b1803f49d1ca"
-					(reference "#PWR057")
+					(reference "#PWR055")
 					(unit 1)
 				)
@@
 		(on_board yes)
 		(dnp no)
-		(property "Reference" "J4"
+		(property "Reference" "J5"
 			(at 206.756 91.44 0)
 			(effects
@@
 			(project "XMOS_demo"
 				(path "/0a855fb0-ca19-4770-811e-70d8770d7fdd/82ce7187-f0cb-4a8a-9f6c-b1803f49d1ca"
-					(reference "J4")
+					(reference "J5")
 					(unit 1)
 				)
@@
 		(on_board yes)
 		(dnp no)
-		(property "Reference" "R29"
+		(property "Reference" "R27"
 			(at 113.538 57.404 0)
 			(effects
@@
 			(project "XMOS_demo"
 				(path "/0a855fb0-ca19-4770-811e-70d8770d7fdd/82ce7187-f0cb-4a8a-9f6c-b1803f49d1ca"
-					(reference "R29")
+					(reference "R27")
 					(unit 1)
 				)
@@
 		(on_board yes)
 		(dnp yes)
-		(property "Reference" "R34"
+		(property "Reference" "R32"
 			(at 195.834 98.044 0)
 			(effects
@@
 			(project "XMOS_demo"
 				(path "/0a855fb0-ca19-4770-811e-70d8770d7fdd/82ce7187-f0cb-4a8a-9f6c-b1803f49d1ca"
-					(reference "R34")
+					(reference "R32")
 					(unit 1)
 				)
@@
 		(on_board yes)
 		(dnp no)
-		(property "Reference" "R31"
+		(property "Reference" "R29"
 			(at 109.22 87.376 90)
 			(effects
@@
 			(project "XMOS_demo"
 				(path "/0a855fb0-ca19-4770-811e-70d8770d7fdd/82ce7187-f0cb-4a8a-9f6c-b1803f49d1ca"
-					(reference "R31")
+					(reference "R29")
 					(unit 1)
 				)
@@
 		(on_board yes)
 		(dnp no)
-		(property "Reference" "#PWR059"
+		(property "Reference" "#PWR057"
 			(at 116.84 82.55 0)
 			(effects
@@
 			(project "XMOS_demo"
 				(path "/0a855fb0-ca19-4770-811e-70d8770d7fdd/82ce7187-f0cb-4a8a-9f6c-b1803f49d1ca"
-					(reference "#PWR059")
+					(reference "#PWR057")
 					(unit 1)
 				)
@@
 		(on_board yes)
 		(dnp no)
-		(property "Reference" "R30"
+		(property "Reference" "R28"
 			(at 114.3 84.836 90)
 			(effects
@@
 			(project "XMOS_demo"
 				(path "/0a855fb0-ca19-4770-811e-70d8770d7fdd/82ce7187-f0cb-4a8a-9f6c-b1803f49d1ca"
-					(reference "R30")
+					(reference "R28")
 					(unit 1)
 				)
@@
 		(on_board yes)
 		(dnp no)
-		(property "Reference" "R33"
+		(property "Reference" "R31"
 			(at 109.22 92.456 90)
 			(effects
@@
 			(project "XMOS_demo"
 				(path "/0a855fb0-ca19-4770-811e-70d8770d7fdd/82ce7187-f0cb-4a8a-9f6c-b1803f49d1ca"
-					(reference "R33")
+					(reference "R31")
 					(unit 1)
 				)
@@
 		(on_board yes)
 		(dnp no)
-		(property "Reference" "#PWR064"
+		(property "Reference" "#PWR062"
 			(at 144.78 133.35 0)
 			(effects
@@
 			(project "XMOS_demo"
 				(path "/0a855fb0-ca19-4770-811e-70d8770d7fdd/82ce7187-f0cb-4a8a-9f6c-b1803f49d1ca"
-					(reference "#PWR064")
+					(reference "#PWR062")
 					(unit 1)
 				)
@@
 		(dnp no)
 		(fields_autoplaced yes)
-		(property "Reference" "#PWR062"
+		(property "Reference" "#PWR060"
 			(at 124.46 110.49 0)
 			(effects
@@
 			(project "XMOS_demo"
 				(path "/0a855fb0-ca19-4770-811e-70d8770d7fdd/82ce7187-f0cb-4a8a-9f6c-b1803f49d1ca"
-					(reference "#PWR062")
+					(reference "#PWR060")
 					(unit 1)
 				)
@@
 		(on_board yes)
 		(dnp yes)
-		(property "Reference" "R35"
+		(property "Reference" "R33"
 			(at 127.508 110.744 0)
 			(effects
@@
 			(project "XMOS_demo"
 				(path "/0a855fb0-ca19-4770-811e-70d8770d7fdd/82ce7187-f0cb-4a8a-9f6c-b1803f49d1ca"
-					(reference "R35")
+					(reference "R33")
+					(unit 1)
+				)
+			)
+		)
+	)
+	(symbol
+		(lib_id "power:PWR_FLAG")
+		(at 132.08 60.96 0)
+		(unit 1)
+		(exclude_from_sim no)
+		(in_bom yes)
+		(on_board yes)
+		(dnp no)
+		(fields_autoplaced yes)
+		(property "Reference" "#FLG06"
+			(at 132.08 59.055 0)
+			(effects
+				(font
+					(size 1.27 1.27)
+				)
+				(hide yes)
+			)
+		)
+		(property "Value" "PWR_FLAG"
+			(at 132.08 55.88 0)
+			(effects
+				(font
+					(size 1.27 1.27)
+				)
+			)
+		)
+		(property "Footprint" ""
+			(at 132.08 60.96 0)
+			(effects
+				(font
+					(size 1.27 1.27)
+				)
+				(hide yes)
+			)
+		)
+		(property "Datasheet" "~"
+			(at 132.08 60.96 0)
+			(effects
+				(font
+					(size 1.27 1.27)
+				)
+				(hide yes)
+			)
+		)
+		(property "Description" "Special symbol for telling ERC where power comes from"
+			(at 132.08 60.96 0)
+			(effects
+				(font
+					(size 1.27 1.27)
+				)
+				(hide yes)
+			)
+		)
+		(pin "1"
+		)
+		(instances
+			(project "XMOS_demo"
+				(path "/0a855fb0-ca19-4770-811e-70d8770d7fdd/82ce7187-f0cb-4a8a-9f6c-b1803f49d1ca"
+					(reference "#FLG06")
 					(unit 1)
 				)
@@
 		(on_board yes)
 		(dnp no)
-		(property "Reference" "#PWR060"
+		(property "Reference" "#PWR058"
 			(at 200.66 95.25 0)
 			(effects
@@
 			(project "XMOS_demo"
 				(path "/0a855fb0-ca19-4770-811e-70d8770d7fdd/82ce7187-f0cb-4a8a-9f6c-b1803f49d1ca"
-					(reference "#PWR060")
+					(reference "#PWR058")
 					(unit 1)
 				)
@@
 		(on_board yes)
 		(dnp no)
-		(property "Reference" "#PWR063"
+		(property "Reference" "#PWR061"
 			(at 167.64 125.73 0)
 			(effects
@@
 			(project "XMOS_demo"
 				(path "/0a855fb0-ca19-4770-811e-70d8770d7fdd/82ce7187-f0cb-4a8a-9f6c-b1803f49d1ca"
-					(reference "#PWR063")
+					(reference "#PWR061")
 					(unit 1)
 				)

Commit message: sch work changes (jumpers, connectors, tp)
Parts:
- added J9: Conn_01x06_Socket, Connector_PinHeader_2.54mm:PinHeader_1x06_P2.54mm_Vertical, symbol Connector:Conn_01x06_Socket
Connections:
- net GND: now also J9.6 (Pin_6)
- net INL+: now also J9.4 (Pin_4)
- net INL-: now also J9.5 (Pin_5)
- net INR+: now also J9.2 (Pin_2)
- net INR-: now also J9.3 (Pin_3)
- net P5V0: now also J9.1 (Pin_1)
Other:
- moved on the sheet: C31, C32, C33, C34, C35, C36, C37, C38, C39, C40, C41, C42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

Commit message: Summary (required)
Parts:
- removed R34: 0R, Resistor_SMD:R_0603_1608Metric, symbol Device:R_Small
- renumbered C31 to C39, C32 to C40, C33 to C41, C34 to C42, C35 to C43, C36 to C44, C37 to C45, C38 to C46, C39 to C47, C40 to C48, C41 to C49, C42 to C50, C43 to C51, C44 to C52, J9 to J6, R27 to R35, R28 to R36, R29 to R37, R30 to R38, R31 to R39, R32 to R40, R33 to R41
Connections:
- net ~{SHDN}: now also R41.2, U7.16 (~{SHDN})

Commit message: Started changes on power supply (audio in) on schematic
Parts:
- renumbered C44 to C40, C46 to C41, C48 to C42, C45 to C44, C47 to C45, C49 to C46, C40 to C47, C41 to C48, C42 to C49, C51 to C50, C52 to C51, C50 to C52, J6 to J5, J5 to J6, R37 to R36, R39 to R37, R36 to R38, R38 to R39, R35 to R40, R40 to R42
