File: XMOS_demo/XMOS_demo.kicad_pcb (KiCad board)
At the start: 2 copper layers, 100 x 100 mm, 170 parts, among them J1 XSYS2 DEBUG CONNECTOR, J2 Screw_Terminal, J3 Conn_01x02_Pin, J4 USB_C_Receptacle_USB2.0_16P, J5 AudioJack3_SwitchT, J6 AudioJack2_SwitchT, J7 AudioJack2_SwitchT, U1 U316-1024-QF60B, U10 OPA340NA, U11 OPA340NA, U2 W25Q32JVSS, U3 TPD3S014, U4 TLV75733PDBV, U5 TLV75718PDBV, U6 AP61200Z6, U7 MAX97220C, U8 CS4271, U9 OPA340NA, Y1 Crystal_24M, Y2 24.576M

Commit message: merge
Parts:
- C46, C48, C49: footprint Capacitor_SMD:C_0603_1608Metric -> Capacitor_SMD:C_0402_1005Metric
- moved C52 31.0 mm to (114.8, 135.9), turned to 90 degrees
- moved C55 29.6 mm to (133.9, 141.8), turned to -90 degrees
- moved Y2 26.1 mm to (131.4, 141.8), turned to 0 degrees
- moved C51 24.9 mm to (122.3, 137.7), turned to 90 degrees
- moved R35 24.6 mm to (119.5, 134.7), turned to -90 degrees
- moved R38 24.6 mm to (138.8, 139.8), turned to 180 degrees
- moved C64 23.1 mm to (116.8, 124.4), turned to -90 degrees
- moved C50 23.0 mm to (121.0, 134.7), turned to -90 degrees
- moved R40 22.7 mm to (138.8, 138.3), turned to 180 degrees
- moved C56 22.5 mm to (128.9, 141.8), turned to 90 degrees
- moved C49 21.5 mm to (122.5, 134.7), turned to -90 degrees
- moved R41 20.9 mm to (138.8, 136.8), turned to 180 degrees
- moved C58 20.8 mm to (119.3, 128.9), turned to 90 degrees
- moved R42 20.4 mm to (139.8, 135.3), turned to 180 degrees
- moved R46 20.4 mm to (127.5, 141.8), turned to -90 degrees
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Connections:
- U1 pad 48: /MCU/LED3 -> /MCU/LED2
- U1 pad 50: /MCU/LED2 -> /MCU/LED3
Routing:
- net /Codec/MCLK: track 0.00 -> 55.6 mm, vias 0 -> 2
- net /MCU/I2S_SCLK: track 0.00 -> 48.8 mm, vias 0 -> 2
- net /MCU/I2S_LRCK: track 0.00 -> 47.6 mm, vias 0 -> 1
- net /MCU/I2S_DAC: track 0.00 -> 27.1 mm
- net /MCU/I2S_ADC: track 0.00 -> 24.7 mm
- net /Codec/SDA: track 2.62 -> 15.6 mm
- net /Codec/SCL: track 6.86 -> 19.1 mm
- net P3V3: track 14.0 -> 26.1 mm, vias 6 -> 7
- net /MCU/LED1: track 1.84 -> 10.3 mm
- net /MCU/LED3: track 1.82 -> 9.99 mm
- net /MCU/LED2: track 1.82 -> 9.99 mm
- net /Codec/SDIN: track 0.00 -> 7.98 mm
- net /Codec/SDOUT: track 0.00 -> 7.75 mm
- net /Codec/LRCK: track 0.00 -> 7.42 mm
- net /Codec/SCLK: track 0.00 -> 7.07 mm
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- added copper zone on B.Cu, net GND
- added copper zone on In1.Cu, net GND
- added copper zone on In2.Cu, net GND
- added copper zone on B.Cu, net P0V9
Other:
- copper layers 2 -> 4

Commit message: pcb routing
Parts:
- removed NT1, NT2, NT3, NT4, NT5: NetTie_2, NetTie:NetTie-2_SMD_Pad0.5mm
- added D5: LED, LED_SMD:LED_0603_1608Metric, F.Cu at (137.4, 148.9)
- added D6: LED, LED_SMD:LED_0603_1608Metric, F.Cu at (138.9, 148.9)
- added J8: Conn_01x06_Socket, Connector_PinHeader_2.54mm:PinHeader_1x06_P2.54mm_Vertical, F.Cu at (126.7, 109.0)
- added J9: Conn_01x06_Socket, Connector_PinHeader_2.54mm:PinHeader_1x06_P2.54mm_Vertical, F.Cu at (122.5, 96.8)
- added R24: 1k, Resistor_SMD:R_0603_1608Metric, F.Cu at (137.4, 145.9)
- added R26: 1k, Resistor_SMD:R_0603_1608Metric, F.Cu at (138.9, 145.9)
- added R53: 0R, Resistor_SMD:R_0603_1608Metric, F.Cu at (159.6, 134.5)
- added R54: 0R, Resistor_SMD:R_0603_1608Metric, F.Cu at (185.9, 137.3)
- added R55: 0R, Resistor_SMD:R_0603_1608Metric, F.Cu at (181.2, 142.9)
- added R56: 0R, Resistor_SMD:R_0603_1608Metric, F.Cu at (101.3, 80.8)
- added R57: 0R, Resistor_SMD:R_0603_1608Metric, F.Cu at (117.3, 102.7)
- added R58: 0R, Resistor_SMD:R_0603_1608Metric, F.Cu at (115.7, 102.7)
- added R59: 0R, Resistor_SMD:R_0603_1608Metric, F.Cu at (114.1, 102.7)
- added R60: 0R, Resistor_SMD:R_0603_1608Metric, F.Cu at (112.4, 102.7)
- added TP10: TestPoint, TestPoint:TestPoint_Pad_D2.0mm, F.Cu at (183.7, 135.8)
- added TP11: TestPoint, TestPoint:TestPoint_Pad_D2.0mm, F.Cu at (178.1, 143.8)
- R1, R2, R3: value 680R -> 1k
- moved C35 18.1 mm to (119.8, 87.8)
- moved C39 18.1 mm to (117.3, 90.2)
- moved C36 14.2 mm to (105.2, 87.8)
- moved C37 9.94 mm to (101.1, 87.8)
- moved C40 9.94 mm to (108.1, 90.2)
- moved C41 9.94 mm to (98.6, 90.2)
- moved C31 7.90 mm to (123.8, 87.8)
- moved C38 7.61 mm to (126.7, 90.2)
- moved TP8 4.65 mm to (179.4, 131.4)
- moved R30 4.34 mm to (104.8, 77.1)
- moved R31 4.34 mm to (104.8, 75.6)
- moved RN2 4.34 mm to (103.3, 71.4)
- moved R33 4.33 mm to (104.5, 80.8)
- moved R34 4.33 mm to (103.0, 80.8)
- moved C32 3.45 mm to (111.3, 79.1)
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Connections:
- net /Audio In/VQ2 renamed /Audio In/VQ2_3
- C24 pad 1: P5V0 -> Net-(U4-IN)
- C26 pad 1: P5V0 -> Net-(U5-IN)
- C30 pad 1: P5V0 -> Net-(U6-VIN)
- R20 pad 1: P5V0 -> Net-(U4-IN)
- R21 pad 1: P5V0 -> Net-(U5-IN)
- R22 pad 1: P5V0 -> Net-(U6-VIN)
- TP5 pad 1: P5V0 -> Net-(U4-IN)
- U1 pad 48: /MCU/LED2 -> /MCU/LED3
- U1 pad 50: /MCU/LED3 -> /MCU/LED2
- U4 pad 1: P5V0 -> Net-(U4-IN)
- U5 pad 1: P5V0 -> Net-(U5-IN)
- U6 pad 3: P5V0 -> Net-(U6-VIN)
Routing:
- net /MCU/I2S_ADC: track 24.7 -> 53.9 mm, vias 0 -> 2
- net /MCU/I2S_DAC: track 27.1 -> 53.3 mm, vias 0 -> 2
- net Net-(U4-IN): track 0.00 -> 9.59 mm
- net P5V0: track 9.62 -> 0.05 mm, vias 4 -> 3
- net /MCU/I2S_LRCK: track 47.6 -> 54.3 mm, vias 1 -> 2
- net /MCU/CODEC_~{RST}: track 0.00 -> 6.33 mm, vias 0 -> 1
- net Net-(U6-VIN): track 0.00 -> 4.68 mm
- net P3V3: track 26.1 -> 29.3 mm
- net P1V8: track 12.6 -> 15.8 mm
- net Net-(J2-Pin_2): track 6.85 -> 9.10 mm
- net GND: track 32.6 -> 32.0 mm
- net P0V9: track 29.5 -> 29.9 mm, vias 7 -> 9

Commit message: Summary (required)
Parts:
- removed the R34 at (103.0, 80.8)
- added J10: Conn_PMOD_02x06, _Connector:PMOD_PinHeader_2x06_P2.54mm_Horizontal, F.Cu at (53.8, 86.7)
- added J11: Conn_PMOD_02x06, _Connector:PMOD_PinHeader_2x06_P2.54mm_Horizontal, F.Cu at (54.2, 104.2)
- added JP1: Jumper_3_Bridged12, Connector_PinHeader_2.54mm:PinHeader_1x03_P2.54mm_Vertical, F.Cu at (70.5, 75.7)
- added JP10: Jumper_3_Bridged12, Connector_PinHeader_2.54mm:PinHeader_1x03_P2.54mm_Vertical, F.Cu at (71.4, 89.3)
- added JP2: Jumper_3_Bridged12, Connector_PinHeader_2.54mm:PinHeader_1x03_P2.54mm_Vertical, F.Cu at (75.5, 79.6)
- added JP3: Jumper_3_Bridged12, Connector_PinHeader_2.54mm:PinHeader_1x03_P2.54mm_Vertical, F.Cu at (71.3, 97.7)
- added JP4: Jumper_3_Bridged12, Connector_PinHeader_2.54mm:PinHeader_1x03_P2.54mm_Vertical, F.Cu at (71.5, 101.5)
- added JP5: Jumper_3_Bridged12, Connector_PinHeader_2.54mm:PinHeader_1x03_P2.54mm_Vertical, F.Cu at (71.4, 110.5)
- added JP6: Jumper_3_Bridged12, Connector_PinHeader_2.54mm:PinHeader_1x03_P2.54mm_Vertical, F.Cu at (71.4, 114.5)
- added JP7: Jumper_3_Bridged12, Connector_PinHeader_2.54mm:PinHeader_1x03_P2.54mm_Vertical, F.Cu at (75.3, 64.6)
- added JP8: Jumper_3_Bridged12, Connector_PinHeader_2.54mm:PinHeader_1x03_P2.54mm_Vertical, F.Cu at (75.2, 68.8)
- added JP9: Jumper_3_Bridged12, Connector_PinHeader_2.54mm:PinHeader_1x03_P2.54mm_Vertical, F.Cu at (71.4, 85.4)
- renumbered C66 to C1, C3 to C10, C4 to C11, C5 to C12, C6 to C13, C7 to C14, C8 to C15, C9 to C16, C10 to C17, C11 to C18, C12 to C19, C67 to C2, C13 to C20, C14 to C21, C15 to C22, C16 to C23, C17 to C24, C1 to C25, C18 to C26, C19 to C27, C20 to C28, C21 to C29, C68 to C3, C22 to C30, C23 to C31, C24 to C32, C25 to C33, C26 to C34, C27 to C35, C28 to C36, C29 to C37, C30 to C38, C31 to C39, C69 to C4, C32 to C40, C33 to C41, C34 to C42, C35 to C43, C36 to C44, C37 to C45, C38 to C46, C39 to C47, C40 to C48, C41 to C49, C70 to C5, C42 to C50, C43 to C51, C44 to C52, C45 to C53, C46 to C54, C47 to C55, C48 to C56, C49 to C57, C50 to C58, C51 to C59, C71 to C6, C52 to C60, C53 to C61, C54 to C62, C55 to C63, C56 to C64, C57 to C65, C58 to C66, C59 to C67, C60 to C68, C61 to C69, C72 to C7, C62 to C70, C63 to C71, C64 to C72, C65 to C73, C73 to C8, C2 to C9, J9 to J6, J8 to J7, J6 to J8, J7 to J9, R57 to R1, R5 to R10, R6 to R11, R7 to R12, R8 to R13, R9 to R14, R10 to R15, R11 to R16, R12 to R17, R13 to R18, R14 to R19, R58 to R2, R15 to R20, R16 to R21, R17 to R22, R24 to R23, R26 to R24, R18 to R25, R19 to R26, R53 to R27, R20 to R28, R54 to R29, R59 to R3, R21 to R30, R55 to R31, R22 to R32, R23 to R33, R25 to R34, R27 to R35, R28 to R36, R29 to R37, R30 to R38, R31 to R39, R60 to R4, R32 to R40, R33 to R41, R35 to R42, R36 to R43, R37 to R44, R38 to R45, R39 to R46, R40 to R47, R41 to R48, R42 to R49, R56 to R5, R43 to R50, R44 to R51, R45 to R52, R46 to R53, R47 to R54, R48 to R55, R49 to R56, R50 to R57, R51 to R58, R52 to R59, R4 to R6, R1 to R7, R2 to R8, R3 to R9, TP8 to TP10, TP9 to TP11, TP10 to TP7, TP7 to TP8, TP11 to TP9
Connections:
- R41 pad 2: Net-(U7-~{SHDN}) -> /Audio Out/~{SHDN}
- R45 pad 1: /Codec/MCLK -> /Codec/MCLK_IN
- R47 pad 1: /MCU/I2S_LRCK -> /Codec/I2S_LRCK_IN
- R48 pad 1: /MCU/I2S_SCLK -> /Codec/I2S_SCLK_IN
- R49 pad 1: /MCU/I2S_ADC -> /Codec/I2S_ADC_OUT
- R50 pad 1: /MCU/I2S_DAC -> /Codec/I2S_DAC_IN
- U1 pad 10: /MCU/I2S_LRCK -> /MCU/I2S_LRCK_OUT
- U1 pad 13: /MCU/I2S_SCLK -> /MCU/I2S_SCLK_OUT
- U1 pad 14: /Codec/MCLK -> /MCU/MCLK_OUT
- U1 pad 7: /MCU/I2S_ADC -> /MCU/I2S_ADC_IN
- U1 pad 9: /MCU/I2S_DAC -> /MCU/I2S_DAC_OUT
- U7 pad 16: Net-(U7-~{SHDN}) -> /Audio Out/~{SHDN}
Routing:
- net (no net): track 0.00 -> 209.9 mm, vias 0 -> 8
- net /MCU/I2S_LRCK: track 54.3 -> 0.00 mm, vias 2 -> 0
- net /MCU/I2S_ADC: track 53.9 -> 0.00 mm, vias 2 -> 0
- net /MCU/I2S_DAC: track 53.3 -> 0.00 mm, vias 2 -> 0
- net /MCU/I2S_SCLK: track 48.4 -> 0.00 mm, vias 2 -> 0

Commit message: PCB work
Parts:
- removed the C61 at (128.0, 125.3)
- removed the C62 at (124.5, 123.5)
- removed the J7 at (126.7, 109.0)
- removed the R1 at (117.3, 102.7)
- removed the R2 at (115.7, 102.7)
- removed the R3 at (114.1, 102.7)
- removed the R4 at (112.4, 102.7)
- removed the R5 at (101.3, 80.8)
- added C30: 100u, Capacitor_SMD:CP_Elec_6.3x5.7, F.Cu at (184.4, 138.3)
- added C31: 100u, Capacitor_SMD:CP_Elec_6.3x5.7, F.Cu at (143.6, 132.3)
- added C46: 2n7, Capacitor_SMD:C_0603_1608Metric, F.Cu at (119.9, 96.4)
- added C49: 470p, Capacitor_SMD:C_0603_1608Metric, F.Cu at (118.4, 97.9)
- added C53: 2n7, Capacitor_SMD:C_0603_1608Metric, F.Cu at (116.8, 96.4)
- added C57: 2n7, Capacitor_SMD:C_0603_1608Metric, F.Cu at (110.3, 95.9)
- added C59: 470p, Capacitor_SMD:C_0603_1608Metric, F.Cu at (108.5, 98.0)
- added C60: 2n7, Capacitor_SMD:C_0603_1608Metric, F.Cu at (106.5, 95.7)
- added C74: 1u, Capacitor_SMD:CP_Elec_4x5.4, F.Cu at (146.0, 105.2)
- added C75: 100n, Capacitor_SMD:C_0603_1608Metric, F.Cu at (142.1, 102.8)
- added C78: 1u, Capacitor_SMD:C_0603_1608Metric, F.Cu at (142.7, 91.8)
- added C80: 1u, Capacitor_SMD:C_0603_1608Metric, F.Cu at (142.7, 96.3)
- added C82: 1u, Capacitor_SMD:C_0603_1608Metric, F.Cu at (161.4, 74.6)
- added C84: 1u, Capacitor_SMD:C_0603_1608Metric, F.Cu at (152.8, 71.5)
- added C86: 1u, Capacitor_SMD:C_0603_1608Metric, F.Cu at (172.9, 71.5)
- added J5: Conn_01x06_Socket, Connector_PinHeader_2.54mm:PinHeader_1x06_P2.54mm_Vertical, F.Cu at (121.1, 103.1)
- added R17: 0R, Resistor_SMD:R_0603_1608Metric, F.Cu at (151.6, 140.3)
- added R32: 634R, Resistor_SMD:R_0603_1608Metric, F.Cu at (120.9, 99.1)
- added R34: 634R, Resistor_SMD:R_0603_1608Metric, F.Cu at (115.9, 99.2)
- added R40: 0R, Resistor_SMD:R_0603_1608Metric, F.Cu at (127.7, 104.0)
- added R41: 634R, Resistor_SMD:R_0603_1608Metric, F.Cu at (111.2, 98.8)
- added R42: 634R, Resistor_SMD:R_0603_1608Metric, F.Cu at (105.9, 98.9)
- added R59: 0R, Resistor_SMD:R_0603_1608Metric, F.Cu at (143.4, 94.0)
- added R61: 0R, Resistor_SMD:R_0603_1608Metric, F.Cu at (161.4, 71.6)
- added TP5: TestPoint, TestPoint:TestPoint_Keystone_5005-5009_Compact, F.Cu at (146.6, 141.4)
- added TP6: TestPoint, TestPoint:TestPoint_Keystone_5005-5009_Compact, F.Cu at (140.5, 141.8)
- C73: renamed from C67; value 1u -> 10u
- C77: renamed from C69; value 1u -> 10u
- R16: renamed from R21; value 0R3 -> 0R
- moved C85 76.0 mm to (171.4, 71.5), turned to 90 degrees
- moved J10 69.1 mm to (98.5, 139.3)
- moved JP7 62.1 mm to (109.8, 116.2)
- moved JP1 62.1 mm to (109.8, 123.7), turned to -90 degrees
- moved JP9 59.7 mm to (109.8, 131.1)
- moved JP3 56.3 mm to (109.8, 138.8)
- moved JP8 55.8 mm to (109.8, 112.6)
- moved JP10 54.1 mm to (109.8, 127.5)
- moved JP2 53.0 mm to (109.8, 120.0)
- moved JP5 52.6 mm to (109.8, 146.4)
- moved JP4 51.0 mm to (109.8, 135.2)
- moved JP6 47.8 mm to (109.8, 142.8)
- moved J11 46.0 mm to (98.5, 116.4)
- moved C68 43.8 mm to (132.7, 96.0), turned to 0 degrees
- moved R43 37.4 mm to (134.8, 100.5), turned to 180 degrees
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- renumbered C30 to C32, C31 to C33, C32 to C34, C33 to C35, C34 to C36, C35 to C37, C36 to C38, C37 to C39, C38 to C40, C39 to C41, C40 to C42, C41 to C43, C42 to C44, C43 to C45, C44 to C47, C45 to C48, C46 to C50, C47 to C51, C48 to C52, C49 to C54, C50 to C55, C51 to C56, C52 to C58, C53 to C61, C54 to C62, C55 to C63, C56 to C64, C57 to C65, C58 to C66, C59 to C67, C60 to C68, C63 to C69, C64 to C70, C65 to C71, C66 to C72, C68 to C76, C73 to C79, C70 to C81, C71 to C83, C72 to C85, J5 to J7, R6 to R1, R15 to R10, R16 to R11, R17 to R12, R18 to R13, R19 to R14, R20 to R15, R22 to R18, R23 to R19, R7 to R2, R24 to R20, R25 to R21, R26 to R22, R27 to R23, R28 to R24, R29 to R25, R30 to R26, R31 to R27, R32 to R28, R33 to R29, R8 to R3, R34 to R30, R35 to R31, R36 to R33, R37 to R35, R38 to R36, R39 to R37, R40 to R38, R41 to R39, R9 to R4, R42 to R43, R43 to R44, R44 to R45, R45 to R46, R46 to R47, R47 to R48, R48 to R49, R10 to R5, R49 to R50, R50 to R51, R51 to R52, R52 to R53, R53 to R54, R54 to R55, R55 to R56, R56 to R57, R57 to R58, R11 to R6, R58 to R60, R59 to R62, R12 to R7, R13 to R8, R14 to R9, TP8 to TP10, TP9 to TP11, TP10 to TP12, TP11 to TP13, TP5 to TP7, TP6 to TP8, TP7 to TP9
Connections:
- net /Audio Out/~{SHDN} renamed Net-(U7-~{SHDN})
- C79 pad 1: P5V0 -> P_OP2_SUPPLY
- C83 pad 1: P5V0 -> P_OP1_SUPPLY
- C85 pad 1: P5V0 -> P_OP1_SUPPLY
- J4 pad A4: VBUS -> Net-(J4-VBUS-PadA4)
- J4 pad A9: VBUS -> Net-(J4-VBUS-PadA4)
- J4 pad B4: VBUS -> Net-(J4-VBUS-PadA4)
- J4 pad B9: VBUS -> Net-(J4-VBUS-PadA4)
- R2 pad 1: /MCU/LED3 -> /MCU/LED1
- R4 pad 1: /MCU/LED1 -> /MCU/LED3
- U1 pad 46: /MCU/LED1 -> /MCU/LED3
- U1 pad 48: /MCU/LED3 -> /MCU/LED2
- U1 pad 50: /MCU/LED2 -> /MCU/LED1
- U10 pad 5: P5V0 -> P_OP2_SUPPLY
- U11 pad 5: P5V0 -> P_OP1_SUPPLY
- U8 pad 23: /Codec/~{MUTE} -> /Audio Out/~{MUTE}
- U8 pad 24: /Codec/OUT_A- -> /Audio Out/OUT_A-
- U8 pad 25: /Codec/OUT_A+ -> /Audio Out/OUT_A+
- U8 pad 26: /Codec/OUT_B+ -> /Audio Out/OUT_B+
- U8 pad 27: /Codec/OUT_B- -> /Audio Out/OUT_B-
- U9 pad 5: P5V0 -> P_OP1_SUPPLY
Routing:
- net (no net): track 209.9 -> 0.00 mm, vias 8 -> 0
- net /Codec/MCLK: track 55.9 -> 7.77 mm, vias 2 -> 0
- net /MCU/I2S_LRCK_OUT: track 0.00 -> 18.1 mm, vias 0 -> 1
- net /MCU/I2S_DAC_OUT: track 0.00 -> 17.6 mm, vias 0 -> 1
- net /MCU/I2S_ADC_IN: track 0.00 -> 17.0 mm, vias 0 -> 1
- net /MCU/MCLK_OUT: track 0.00 -> 16.5 mm, vias 0 -> 1
- net /I2S_Confing/I2S_SCLK_PMOD1: track 0.00 -> 15.8 mm
- net /MCU/I2S_SCLK_OUT: track 0.00 -> 14.4 mm, vias 0 -> 1
- net /I2S_Confing/MCLK_PMOD1: track 0.00 -> 13.3 mm
- net Net-(J4-VBUS-PadA4): track 0.00 -> 13.1 mm
- net /I2S_Confing/I2S_LRCK_PMOD1: track 0.00 -> 13.0 mm
- net /I2S_Confing/I2S_ADC_PMOD1: track 0.00 -> 10.7 mm
- net Net-(U5-IN): track 0.04 -> 8.02 mm
- net /Codec/SCL: track 19.1 -> 12.0 mm
- net /Codec/SDA: track 15.6 -> 8.54 mm
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- added copper zone on F.Cu, net VBUS
