File: XMOS_demo/codec.kicad_sch (KiCad schematic)
At the start: 27 parts, among them J8 Conn_01x06_Socket, U8 CS4271, Y2 24.576M

Commit message: Summary (required)
Parts:
- renumbered C45 to C53, C46 to C54, C47 to C55, C48 to C56, C49 to C57, C50 to C58, C51 to C59, C52 to C60, C53 to C61, C54 to C62, C55 to C63, C56 to C64, J8 to J7, R35 to R42, R36 to R43, R37 to R44, R38 to R45, R39 to R46, R40 to R47, R41 to R48, R42 to R49, R43 to R50, R44 to R51, R45 to R52, R46 to R53

Commit message: Started changes on power supply (audio in) on schematic
Parts:
- renumbered C63 to C53, C53 to C54, C54 to C55, C64 to C56, C55 to C57, C56 to C58, C57 to C59, C58 to C60, C59 to C63, C60 to C64, R49 to R44, R46 to R45, R52 to R46, R44 to R47, R51 to R48, R47 to R49, R45 to R50, R48 to R51, R50 to R52, R42 to R54

Commit message: Passive lpf added to autio output
Parts:
- removed C61: 100n, Capacitor_SMD:C_0603_1608Metric, symbol Device:C_Small
- removed C62: 1u, Capacitor_SMD:CP_Elec_4x5.4, symbol Device:C_Polarized_Small
- removed J7: Conn_01x06_Socket, Connector_PinHeader_2.54mm:PinHeader_1x06_P2.54mm_Vertical, symbol Connector:Conn_01x06_Socket
- renumbered C54 to C59, C55 to C60, C57 to C61, C58 to C62, C59 to C63, C60 to C64, C63 to C65, C64 to C66, C53 to C67, C56 to C68, R54 to R43, R43 to R44, R47 to R45, R50 to R46, R45 to R47, R49 to R48, R51 to R49, R44 to R50, R52 to R51, R48 to R52, R46 to R53, R53 to R54
Other:
- moved on the sheet: C59, C60, C61, C62, C63, C64, C65, C66, C67, C68, R43, R44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

Commit message: PCB work
Parts:
- renumbered C59 to C61, C60 to C62, C61 to C63, C62 to C64, C63 to C65, C64 to C66, C65 to C67, C66 to C68, C67 to C69, C68 to C70
Changed lines of the file:
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@@
 		(on_board yes)
 		(dnp yes)
-		(property "Reference" "C67"
+		(property "Reference" "C69"
 			(at 112.776 140.97 0)
 			(effects
@@
 			(project "XMOS_demo"
 				(path "/0a855fb0-ca19-4770-811e-70d8770d7fdd/4b9c48a5-7a99-4cae-9f94-704bf713d5d7"
-					(reference "C67")
+					(reference "C69")
 					(unit 1)
 				)
@@
 		(on_board yes)
 		(dnp no)
-		(property "Reference" "#PWR082"
+		(property "Reference" "#PWR083"
 			(at 210.82 105.41 0)
 			(effects
@@
 			(project "XMOS_demo"
 				(path "/0a855fb0-ca19-4770-811e-70d8770d7fdd/4b9c48a5-7a99-4cae-9f94-704bf713d5d7"
-					(reference "#PWR082")
+					(reference "#PWR083")
 					(unit 1)
 				)
@@
 		(on_board yes)
 		(dnp no)
-		(property "Reference" "#PWR081"
+		(property "Reference" "#PWR082"
 			(at 91.44 102.87 0)
 			(effects
@@
 			(project "XMOS_demo"
 				(path "/0a855fb0-ca19-4770-811e-70d8770d7fdd/4b9c48a5-7a99-4cae-9f94-704bf713d5d7"
-					(reference "#PWR081")
+					(reference "#PWR082")
 					(unit 1)
 				)
@@
 		(on_board yes)
 		(dnp no)
-		(property "Reference" "#PWR084"
+		(property "Reference" "#PWR085"
 			(at 83.82 135.89 0)
 			(effects
@@
 			(project "XMOS_demo"
 				(path "/0a855fb0-ca19-4770-811e-70d8770d7fdd/4b9c48a5-7a99-4cae-9f94-704bf713d5d7"
-					(reference "#PWR084")
+					(reference "#PWR085")
 					(unit 1)
 				)
@@
 		(on_board yes)
 		(dnp yes)
-		(property "Reference" "C68"
+		(property "Reference" "C70"
 			(at 128.524 140.97 0)
 			(effects
@@
 			(project "XMOS_demo"
 				(path "/0a855fb0-ca19-4770-811e-70d8770d7fdd/4b9c48a5-7a99-4cae-9f94-704bf713d5d7"
-					(reference "C68")
+					(reference "C70")
 					(unit 1)
 				)
@@
 		(on_board yes)
 		(dnp no)
-		(property "Reference" "C61"
+		(property "Reference" "C63"
 			(at 135.636 67.31 0)
 			(effects
@@
 			(project "XMOS_demo"
 				(path "/0a855fb0-ca19-4770-811e-70d8770d7fdd/4b9c48a5-7a99-4cae-9f94-704bf713d5d7"
-					(reference "C61")
+					(reference "C63")
 					(unit 1)
 				)
@@
 		(on_board yes)
 		(dnp no)
-		(property "Reference" "C66"
+		(property "Reference" "C68"
 			(at 212.344 90.17 0)
 			(effects
@@
 			(project "XMOS_demo"
 				(path "/0a855fb0-ca19-4770-811e-70d8770d7fdd/4b9c48a5-7a99-4cae-9f94-704bf713d5d7"
-					(reference "C66")
+					(reference "C68")
 					(unit 1)
 				)
@@
 		(on_board yes)
 		(dnp no)
-		(property "Reference" "C65"
+		(property "Reference" "C67"
 			(at 202.184 90.17 0)
 			(effects
@@
 			(project "XMOS_demo"
 				(path "/0a855fb0-ca19-4770-811e-70d8770d7fdd/4b9c48a5-7a99-4cae-9f94-704bf713d5d7"
-					(reference "C65")
+					(reference "C67")
 					(unit 1)
 				)
@@
 		(on_board yes)
 		(dnp no)
-		(property "Reference" "C64"
+		(property "Reference" "C66"
 			(at 174.244 67.31 0)
 			(effects
@@
 			(project "XMOS_demo"
 				(path "/0a855fb0-ca19-4770-811e-70d8770d7fdd/4b9c48a5-7a99-4cae-9f94-704bf713d5d7"
-					(reference "C64")
+					(reference "C66")
 					(unit 1)
 				)
@@
 		(on_board yes)
 		(dnp no)
-		(property "Reference" "C62"
+		(property "Reference" "C64"
 			(at 145.796 67.31 0)
 			(effects
@@
 			(project "XMOS_demo"
 				(path "/0a855fb0-ca19-4770-811e-70d8770d7fdd/4b9c48a5-7a99-4cae-9f94-704bf713d5d7"
-					(reference "C62")
+					(reference "C64")
 					(unit 1)
 				)
@@
 		(on_board yes)
 		(dnp no)
-		(property "Reference" "#PWR076"
+		(property "Reference" "#PWR077"
 			(at 160.02 57.15 0)
 			(effects
@@
 			(project "XMOS_demo"
 				(path "/0a855fb0-ca19-4770-811e-70d8770d7fdd/4b9c48a5-7a99-4cae-9f94-704bf713d5d7"
-					(reference "#PWR076")
+					(reference "#PWR077")
 					(unit 1)
 				)
@@
 		(on_board yes)
 		(dnp no)
-		(property "Reference" "C59"
+		(property "Reference" "C61"
 			(at 115.316 67.31 0)
 			(effects
@@
 			(project "XMOS_demo"
 				(path "/0a855fb0-ca19-4770-811e-70d8770d7fdd/4b9c48a5-7a99-4cae-9f94-704bf713d5d7"
-					(reference "C59")
+					(reference "C61")
 					(unit 1)
 				)
@@
 		(on_board yes)
 		(dnp no)
-		(property "Reference" "C63"
+		(property "Reference" "C65"
 			(at 164.084 67.31 0)
 			(effects
@@
 			(project "XMOS_demo"
 				(path "/0a855fb0-ca19-4770-811e-70d8770d7fdd/4b9c48a5-7a99-4cae-9f94-704bf713d5d7"
-					(reference "C63")
+					(reference "C65")
 					(unit 1)
 				)
@@
 		(on_board yes)
 		(dnp no)
-		(property "Reference" "#PWR080"
+		(property "Reference" "#PWR081"
 			(at 83.82 97.79 0)
 			(effects
@@
 			(project "XMOS_demo"
 				(path "/0a855fb0-ca19-4770-811e-70d8770d7fdd/4b9c48a5-7a99-4cae-9f94-704bf713d5d7"
-					(reference "#PWR080")
+					(reference "#PWR081")
 					(unit 1)
 				)
@@
 		(on_board yes)
 		(dnp no)
-		(property "Reference" "#PWR083"
+		(property "Reference" "#PWR084"
 			(at 91.44 113.03 0)
 			(effects
@@
 			(project "XMOS_demo"
 				(path "/0a855fb0-ca19-4770-811e-70d8770d7fdd/4b9c48a5-7a99-4cae-9f94-704bf713d5d7"
-					(reference "#PWR083")
+					(reference "#PWR084")
 					(unit 1)
 				)
@@
 		(on_board yes)
 		(dnp no)
-		(property "Reference" "#PWR079"
+		(property "Reference" "#PWR080"
 			(at 162.56 82.55 0)
 			(effects
@@
 			(project "XMOS_demo"
 				(path "/0a855fb0-ca19-4770-811e-70d8770d7fdd/4b9c48a5-7a99-4cae-9f94-704bf713d5d7"
-					(reference "#PWR079")
+					(reference "#PWR080")
 					(unit 1)
 				)
@@
 		(on_board yes)
 		(dnp no)
-		(property "Reference" "C60"
+		(property "Reference" "C62"
 			(at 125.476 67.31 0)
 			(effects
@@
 			(project "XMOS_demo"
 				(path "/0a855fb0-ca19-4770-811e-70d8770d7fdd/4b9c48a5-7a99-4cae-9f94-704bf713d5d7"
-					(reference "C60")
+					(reference "C62")
 					(unit 1)
 				)
@@
 		(on_board yes)
 		(dnp no)
-		(property "Reference" "#PWR086"
+		(property "Reference" "#PWR087"
 			(at 157.48 143.51 0)
 			(effects
@@
 			(project "XMOS_demo"
 				(path "/0a855fb0-ca19-4770-811e-70d8770d7fdd/4b9c48a5-7a99-4cae-9f94-704bf713d5d7"
-					(reference "#PWR086")
+					(reference "#PWR087")
 					(unit 1)
 				)
@@
 		(on_board yes)
 		(dnp no)
-		(property "Reference" "#PWR087"
+		(property "Reference" "#PWR088"
 			(at 127 156.21 0)
 			(effects
@@
 			(project "XMOS_demo"
 				(path "/0a855fb0-ca19-4770-811e-70d8770d7fdd/4b9c48a5-7a99-4cae-9f94-704bf713d5d7"
-					(reference "#PWR087")
+					(reference "#PWR088")
 					(unit 1)
 				)
@@
 		(on_board yes)
 		(dnp no)
-		(property "Reference" "#PWR078"
+		(property "Reference" "#PWR079"
 			(at 147.32 82.55 0)
 			(effects
@@
 			(project "XMOS_demo"
 				(path "/0a855fb0-ca19-4770-811e-70d8770d7fdd/4b9c48a5-7a99-4cae-9f94-704bf713d5d7"
-					(reference "#PWR078")
+					(reference "#PWR079")
 					(unit 1)
 				)
@@
 		(on_board yes)
 		(dnp no)
-		(property "Reference" "#PWR077"
+		(property "Reference" "#PWR078"
 			(at 149.86 64.77 0)
 			(effects
@@
 			(project "XMOS_demo"
 				(path "/0a855fb0-ca19-4770-811e-70d8770d7fdd/4b9c48a5-7a99-4cae-9f94-704bf713d5d7"
-					(reference "#PWR077")
+					(reference "#PWR078")
 					(unit 1)
 				)
@@
 		(on_board yes)
 		(dnp no)
-		(property "Reference" "#PWR085"
+		(property "Reference" "#PWR086"
 			(at 137.16 143.51 0)
 			(effects
@@
 			(project "XMOS_demo"
 				(path "/0a855fb0-ca19-4770-811e-70d8770d7fdd/4b9c48a5-7a99-4cae-9f94-704bf713d5d7"
-					(reference "#PWR085")
-					(unit 1)
-				)
+					(reference "#PWR086")
+					(unit 1)
+				)
