File: XMOS_demo/audio_in.kicad_sch (KiCad schematic)
At the start: 29 parts, among them J8 AudioJack2_SwitchT, J9 AudioJack2_SwitchT, U10 OPA340NA, U11 OPA340NA, U9 OPA340NA

Commit message: routing work
Other:
- moved on the sheet: C80
Changed lines of the file:
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@@
 	)
 	(junction
+		(at 53.34 127)
+		(diameter 0)
+		(color 0 0 0 0)
+	)
+	(junction
 		(at 177.8 129.54)
 		(diameter 0)
@@
 	)
 	(junction
+		(at 63.5 127)
+		(diameter 0)
+		(color 0 0 0 0)
+	)
+	(junction
 		(at 55.88 154.94)
 		(diameter 0)
@@
 	)
 	(junction
-		(at 55.88 127)
+		(at 50.8 154.94)
 		(diameter 0)
 		(color 0 0 0 0)
 	)
 	(junction
-		(at 50.8 154.94)
+		(at 66.04 154.94)
 		(diameter 0)
 		(color 0 0 0 0)
@@
 	(wire
 		(pts
-			(xy 55.88 127) (xy 60.96 127)
-		)
-		(stroke
-			(width 0)
-			(type default)
-		)
-	)
-	(wire
-		(pts
 			(xy 152.4 137.16) (xy 152.4 139.7)
 		)
@@
 	(wire
 		(pts
-			(xy 60.96 134.62) (xy 60.96 137.16)
+			(xy 66.04 134.62) (xy 66.04 137.16)
 		)
 		(stroke
@@
 	(wire
 		(pts
+			(xy 66.04 154.94) (xy 71.12 154.94)
+		)
+		(stroke
+			(width 0)
+			(type default)
+		)
+	)
+	(wire
+		(pts
 			(xy 180.34 53.34) (xy 182.88 53.34)
 		)
@@
 	(wire
 		(pts
+			(xy 53.34 127) (xy 63.5 127)
+		)
+		(stroke
+			(width 0)
+			(type default)
+		)
+	)
+	(wire
+		(pts
 			(xy 45.72 154.94) (xy 50.8 154.94)
 		)
@@
 	(wire
 		(pts
-			(xy 50.8 127) (xy 55.88 127)
+			(xy 50.8 127) (xy 53.34 127)
 		)
 		(stroke
@@
 	(wire
 		(pts
+			(xy 63.5 127) (xy 66.04 127)
+		)
+		(stroke
+			(width 0)
+			(type default)
+		)
+	)
+	(wire
+		(pts
 			(xy 205.74 106.68) (xy 205.74 109.22)
 		)
@@
 	(wire
 		(pts
-			(xy 60.96 154.94) (xy 71.12 154.94)
+			(xy 60.96 154.94) (xy 66.04 154.94)
 		)
 		(stroke
@@
 	(wire
 		(pts
-			(xy 55.88 124.46) (xy 55.88 127)
+			(xy 53.34 124.46) (xy 53.34 127)
 		)
 		(stroke
@@
 	(wire
 		(pts
-			(xy 60.96 129.54) (xy 60.96 127)
+			(xy 66.04 129.54) (xy 66.04 127)
 		)
 		(stroke
@@
 	)
 	(symbol
+		(lib_id "power:PWR_FLAG")
+		(at 66.04 154.94 0)
+		(unit 1)
+		(exclude_from_sim no)
+		(in_bom yes)
+		(on_board yes)
+		(dnp no)
+		(property "Reference" "#FLG012"
+			(at 66.04 153.035 0)
+			(effects
+				(font
+					(size 1.27 1.27)
+				)
+				(hide yes)
+			)
+		)
+		(property "Value" "PWR_FLAG"
+			(at 66.04 151.384 0)
+			(effects
+				(font
+					(size 1.016 1.016)
+				)
+			)
+		)
+		(property "Footprint" ""
+			(at 66.04 154.94 0)
+			(effects
+				(font
+					(size 1.27 1.27)
+				)
+				(hide yes)
+			)
+		)
+		(property "Datasheet" "~"
+			(at 66.04 154.94 0)
+			(effects
+				(font
+					(size 1.27 1.27)
+				)
+				(hide yes)
+			)
+		)
+		(property "Description" "Special symbol for telling ERC where power comes from"
+			(at 66.04 154.94 0)
+			(effects
+				(font
+					(size 1.27 1.27)
+				)
+				(hide yes)
+			)
+		)
+		(pin "1"
+		)
+		(instances
+			(project "XMOS_demo"
+				(path "/0a855fb0-ca19-4770-811e-70d8770d7fdd/71bec83b-8ae1-4f4c-8273-5b8329c1423c"
+					(reference "#FLG012")
+					(unit 1)
+				)
+			)
+		)
+	)
+	(symbol
 		(lib_id "_power:P5V0")
 		(at 55.88 152.4 0)
@@
 	(symbol
 		(lib_id "_power:P5V0")
-		(at 55.88 124.46 0)
+		(at 53.34 124.46 0)
 		(unit 1)
 		(exclude_from_sim no)
@@
 		(dnp no)
 		(property "Reference" "#PWR097"
-			(at 55.88 128.27 0)
+			(at 53.34 128.27 0)
 			(effects
 				(font
@@
 		)
 		(property "Value" "P_OP2_SUPPLY"
-			(at 55.88 120.904 0)
+			(at 53.34 120.904 0)
 			(effects
 				(font
@@
 		)
 		(property "Footprint" ""
-			(at 55.88 124.46 0)
+			(at 53.34 124.46 0)
 			(effects
 				(font
@@
 		)
 		(property "Datasheet" ""
-			(at 55.88 124.46 0)
+			(at 53.34 124.46 0)
 			(effects
 				(font
@@
 		)
 		(property "Description" "Power supply for op-amps [2]"
-			(at 55.88 124.46 0)
+			(at 53.34 124.46 0)
 			(effects
 				(font
@@
 	(symbol
 		(lib_id "Device:C_Small")
-		(at 60.96 132.08 0)
+		(at 66.04 132.08 0)
 		(unit 1)
 		(exclude_from_sim no)
@@
 		(dnp no)
 		(property "Reference" "C80"
-			(at 62.484 130.81 0)
+			(at 67.564 130.81 0)
 			(effects
 				(font
@@
 		)
 		(property "Value" "1u"
-			(at 62.484 133.35 0)
+			(at 67.564 133.35 0)
 			(effects
 				(font
@@
 		)
 		(property "Footprint" "Capacitor_SMD:C_0603_1608Metric"
-			(at 60.96 132.08 0)
+			(at 66.04 132.08 0)
 			(effects
 				(font
@@
 		)
 		(property "Datasheet" "~"
-			(at 60.96 132.08 0)
+			(at 66.04 132.08 0)
 			(effects
 				(font
@@
 		)
 		(property "Description" "Unpolarized capacitor, small symbol"
-			(at 60.96 132.08 0)
+			(at 66.04 132.08 0)
 			(effects
 				(font
@@
 		)
 		(property "Dielectirc" "X7R"
-			(at 60.96 132.08 0)
+			(at 66.04 132.08 0)
 			(effects
 				(font
@@
 		)
 		(property "Max Voltage" "16V"
-			(at 60.96 132.08 0)
+			(at 66.04 132.08 0)
 			(effects
 				(font
@@
 	(symbol
 		(lib_id "power:GND")
-		(at 60.96 137.16 0)
+		(at 66.04 137.16 0)
 		(unit 1)
 		(exclude_from_sim no)
@@
 		(dnp no)
 		(property "Reference" "#PWR0101"
-			(at 60.96 143.51 0)
+			(at 66.04 143.51 0)
 			(effects
 				(font
@@
 		)
 		(property "Value" "GND"
-			(at 60.96 140.716 0)
+			(at 66.04 140.716 0)
 			(effects
 				(font
@@
 		)
 		(property "Footprint" ""
-			(at 60.96 137.16 0)
+			(at 66.04 137.16 0)
 			(effects
 				(font
@@
 		)
 		(property "Datasheet" ""
-			(at 60.96 137.16 0)
+			(at 66.04 137.16 0)
 			(effects
 				(font
@@
 		)
 		(property "Description" "Power symbol creates a global label with name \"GND\" , ground"
-			(at 60.96 137.16 0)
+			(at 66.04 137.16 0)
 			(effects
 				(font
@@
 					(unit 1)
 				)
+			)
+		)
+	)
+	(symbol
+		(lib_id "power:PWR_FLAG")
+		(at 63.5 127 0)
+		(unit 1)
+		(exclude_from_sim no)
+		(in_bom yes)
+		(on_board yes)
+		(dnp no)
+		(property "Reference" "#FLG013"
+			(at 63.5 125.095 0)
+			(effects
+				(font
+					(size 1.27 1.27)
+				)
+				(hide yes)
+			)
+		)
+		(property "Value" "PWR_FLAG"
+			(at 63.5 123.444 0)
+			(effects
+				(font
+					(size 1.016 1.016)
+				)
+			)
+		)
+		(property "Footprint" ""
+			(at 63.5 127 0)
+			(effects
+				(font
+					(size 1.27 1.27)
+				)
+				(hide yes)
+			)
+		)
+		(property "Datasheet" "~"
+			(at 63.5 127 0)
+			(effects
+				(font
+					(size 1.27 1.27)
+				)
+				(hide yes)
+			)
+		)
+		(property "Description" "Special symbol for telling ERC where power comes from"
+			(at 63.5 127 0)
+			(effects
+				(font
+					(size 1.27 1.27)
+				)
+				(hide yes)
+			)
+		)
+		(pin "1"
+		)
+		(instances
+			(project "XMOS_demo"
+				(path "/0a855fb0-ca19-4770-811e-70d8770d7fdd/71bec83b-8ae1-4f4c-8273-5b8329c1423c"
+					(reference "#FLG013")
+					(unit 1)
+				)
