File: XMOS_demo/psu.kicad_sch (KiCad schematic)
At the start: 26 parts, among them U4 TLV75733PDBV, U5 TLV75718PDBV, U6 AP61200Z6

Commit message: Summary (required)
Parts:
- renumbered C24 to C32, C25 to C33, C26 to C34, C27 to C35, C28 to C36, C29 to C37, C30 to C38, R53 to R27, R20 to R28, R54 to R29, R21 to R30, R55 to R31, R22 to R32, R23 to R33, R25 to R34, TP8 to TP10, TP9 to TP11, TP10 to TP7, TP7 to TP8, TP11 to TP9

Commit message: Started changes on power supply (audio in) on schematic
Parts:
- renumbered C34 to C33, C38 to C34, C33 to C35, C35 to C36, C36 to C37, C37 to C38, R27 to R28, R31 to R30, R28 to R31, R30 to R32, R32 to R33, R33 to R34, R34 to R35, TP11 to TP10, TP6 to TP11, TP8 to TP12, TP10 to TP13, TP5 to TP7, TP7 to TP8
Other:
- moved on the sheet: TP12

Commit message: Passive lpf added to autio output
Parts:
- renumbered C35 to C33, C33 to C34, C36 to C35, C37 to C36, C38 to C37, C34 to C38, R28 to R23, R31 to R24, R29 to R25, R32 to R26, R30 to R27, R33 to R28, R34 to R29, R35 to R30, TP12 to TP10, TP9 to TP11, TP13 to TP12, TP10 to TP13, TP11 to TP8, TP8 to TP9

Commit message: PCB work
Parts:
- renumbered C32 to C34, C33 to C35, C34 to C36, C35 to C37, C36 to C38, C37 to C39, C38 to C40
Changed lines of the file:
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@@
 		(on_board yes)
 		(dnp no)
-		(property "Reference" "#PWR058"
+		(property "Reference" "#PWR059"
 			(at 157.48 163.83 0)
 			(effects
@@
 			(project "XMOS_demo"
 				(path "/0a855fb0-ca19-4770-811e-70d8770d7fdd/13d4ac51-413b-4f8b-9448-517b4883a5ce"
-					(reference "#PWR058")
+					(reference "#PWR059")
 					(unit 1)
 				)
@@
 		(on_board yes)
 		(dnp no)
-		(property "Reference" "#PWR048"
+		(property "Reference" "#PWR049"
 			(at 91.44 90.17 0)
 			(effects
@@
 			(project "XMOS_demo"
 				(path "/0a855fb0-ca19-4770-811e-70d8770d7fdd/13d4ac51-413b-4f8b-9448-517b4883a5ce"
-					(reference "#PWR048")
+					(reference "#PWR049")
 					(unit 1)
 				)
@@
 		(on_board yes)
 		(dnp no)
-		(property "Reference" "C35"
+		(property "Reference" "C37"
 			(at 131.064 102.87 0)
 			(effects
@@
 			(project "XMOS_demo"
 				(path "/0a855fb0-ca19-4770-811e-70d8770d7fdd/13d4ac51-413b-4f8b-9448-517b4883a5ce"
-					(reference "C35")
+					(reference "C37")
 					(unit 1)
 				)
@@
 		(on_board yes)
 		(dnp yes)
-		(property "Reference" "C36"
+		(property "Reference" "C38"
 			(at 150.876 140.97 0)
 			(effects
@@
 			(project "XMOS_demo"
 				(path "/0a855fb0-ca19-4770-811e-70d8770d7fdd/13d4ac51-413b-4f8b-9448-517b4883a5ce"
-					(reference "C36")
+					(reference "C38")
 					(unit 1)
 				)
@@
 		(on_board yes)
 		(dnp no)
-		(property "Reference" "#PWR046"
+		(property "Reference" "#PWR047"
 			(at 116.84 69.85 0)
 			(effects
@@
 			(project "XMOS_demo"
 				(path "/0a855fb0-ca19-4770-811e-70d8770d7fdd/13d4ac51-413b-4f8b-9448-517b4883a5ce"
-					(reference "#PWR046")
+					(reference "#PWR047")
 					(unit 1)
 				)
@@
 		(on_board yes)
 		(dnp no)
-		(property "Reference" "C33"
+		(property "Reference" "C35"
 			(at 131.064 57.15 0)
 			(effects
@@
 			(project "XMOS_demo"
 				(path "/0a855fb0-ca19-4770-811e-70d8770d7fdd/13d4ac51-413b-4f8b-9448-517b4883a5ce"
-					(reference "C33")
+					(reference "C35")
 					(unit 1)
 				)
@@
 		(on_board yes)
 		(dnp no)
-		(property "Reference" "#PWR053"
+		(property "Reference" "#PWR054"
 			(at 91.44 130.81 0)
 			(effects
@@
 			(project "XMOS_demo"
 				(path "/0a855fb0-ca19-4770-811e-70d8770d7fdd/13d4ac51-413b-4f8b-9448-517b4883a5ce"
-					(reference "#PWR053")
+					(reference "#PWR054")
 					(unit 1)
 				)
@@
 		(on_board yes)
 		(dnp no)
-		(property "Reference" "#PWR044"
+		(property "Reference" "#PWR045"
 			(at 142.24 52.07 0)
 			(effects
@@
 			(project "XMOS_demo"
 				(path "/0a855fb0-ca19-4770-811e-70d8770d7fdd/13d4ac51-413b-4f8b-9448-517b4883a5ce"
-					(reference "#PWR044")
+					(reference "#PWR045")
 					(unit 1)
 				)
@@
 		(on_board yes)
 		(dnp no)
-		(property "Reference" "#PWR055"
+		(property "Reference" "#PWR056"
 			(at 91.44 156.21 0)
 			(effects
@@
 			(project "XMOS_demo"
 				(path "/0a855fb0-ca19-4770-811e-70d8770d7fdd/13d4ac51-413b-4f8b-9448-517b4883a5ce"
-					(reference "#PWR055")
+					(reference "#PWR056")
 					(unit 1)
 				)
@@
 		(on_board yes)
 		(dnp no)
-		(property "Reference" "#PWR050"
+		(property "Reference" "#PWR051"
 			(at 91.44 115.57 0)
 			(effects
@@
 			(project "XMOS_demo"
 				(path "/0a855fb0-ca19-4770-811e-70d8770d7fdd/13d4ac51-413b-4f8b-9448-517b4883a5ce"
-					(reference "#PWR050")
+					(reference "#PWR051")
 					(unit 1)
 				)
@@
 		(on_board yes)
 		(dnp no)
-		(property "Reference" "C38"
+		(property "Reference" "C40"
 			(at 92.964 143.51 0)
 			(effects
@@
 			(project "XMOS_demo"
 				(path "/0a855fb0-ca19-4770-811e-70d8770d7fdd/13d4ac51-413b-4f8b-9448-517b4883a5ce"
-					(reference "C38")
+					(reference "C40")
 					(unit 1)
 				)
@@
 		(on_board yes)
 		(dnp no)
-		(property "Reference" "C34"
+		(property "Reference" "C36"
 			(at 92.964 102.87 0)
 			(effects
@@
 			(project "XMOS_demo"
 				(path "/0a855fb0-ca19-4770-811e-70d8770d7fdd/13d4ac51-413b-4f8b-9448-517b4883a5ce"
-					(reference "C34")
+					(reference "C36")
 					(unit 1)
 				)
@@
 		(on_board yes)
 		(dnp no)
-		(property "Reference" "#PWR043"
+		(property "Reference" "#PWR044"
 			(at 91.44 44.45 0)
 			(effects
@@
 			(project "XMOS_demo"
 				(path "/0a855fb0-ca19-4770-811e-70d8770d7fdd/13d4ac51-413b-4f8b-9448-517b4883a5ce"
-					(reference "#PWR043")
+					(reference "#PWR044")
 					(unit 1)
 				)
@@
 		(on_board yes)
 		(dnp no)
-		(property "Reference" "#PWR054"
+		(property "Reference" "#PWR055"
 			(at 187.96 138.43 0)
 			(effects
@@
 			(project "XMOS_demo"
 				(path "/0a855fb0-ca19-4770-811e-70d8770d7fdd/13d4ac51-413b-4f8b-9448-517b4883a5ce"
-					(reference "#PWR054")
+					(reference "#PWR055")
 					(unit 1)
 				)
@@
 		(on_board yes)
 		(dnp no)
-		(property "Reference" "#PWR047"
+		(property "Reference" "#PWR048"
 			(at 129.54 69.85 0)
 			(effects
@@
 			(project "XMOS_demo"
 				(path "/0a855fb0-ca19-4770-811e-70d8770d7fdd/13d4ac51-413b-4f8b-9448-517b4883a5ce"
-					(reference "#PWR047")
+					(reference "#PWR048")
 					(unit 1)
 				)
@@
 		(on_board yes)
 		(dnp no)
-		(property "Reference" "#PWR056"
+		(property "Reference" "#PWR057"
 			(at 121.92 156.21 0)
 			(effects
@@
 			(project "XMOS_demo"
 				(path "/0a855fb0-ca19-4770-811e-70d8770d7fdd/13d4ac51-413b-4f8b-9448-517b4883a5ce"
-					(reference "#PWR056")
+					(reference "#PWR057")
 					(unit 1)
 				)
@@
 		(on_board yes)
 		(dnp no)
-		(property "Reference" "#PWR051"
+		(property "Reference" "#PWR052"
 			(at 116.84 115.57 0)
 			(effects
@@
 			(project "XMOS_demo"
 				(path "/0a855fb0-ca19-4770-811e-70d8770d7fdd/13d4ac51-413b-4f8b-9448-517b4883a5ce"
-					(reference "#PWR051")
+					(reference "#PWR052")
 					(unit 1)
 				)
@@
 		(on_board yes)
 		(dnp no)
-		(property "Reference" "#PWR045"
+		(property "Reference" "#PWR046"
 			(at 91.44 69.85 0)
 			(effects
@@
 			(project "XMOS_demo"
 				(path "/0a855fb0-ca19-4770-811e-70d8770d7fdd/13d4ac51-413b-4f8b-9448-517b4883a5ce"
-					(reference "#PWR045")
+					(reference "#PWR046")
 					(unit 1)
 				)
@@
 		(on_board yes)
 		(dnp no)
-		(property "Reference" "C32"
+		(property "Reference" "C34"
 			(at 92.964 57.15 0)
 			(effects
@@
 			(project "XMOS_demo"
 				(path "/0a855fb0-ca19-4770-811e-70d8770d7fdd/13d4ac51-413b-4f8b-9448-517b4883a5ce"
-					(reference "C32")
+					(reference "C34")
 					(unit 1)
 				)
@@
 		(on_board yes)
 		(dnp no)
-		(property "Reference" "#PWR049"
+		(property "Reference" "#PWR050"
 			(at 142.24 97.79 0)
 			(effects
@@
 			(project "XMOS_demo"
 				(path "/0a855fb0-ca19-4770-811e-70d8770d7fdd/13d4ac51-413b-4f8b-9448-517b4883a5ce"
-					(reference "#PWR049")
+					(reference "#PWR050")
 					(unit 1)
 				)
@@
 		(on_board yes)
 		(dnp no)
-		(property "Reference" "#PWR052"
+		(property "Reference" "#PWR053"
 			(at 129.54 115.57 0)
 			(effects
@@
 			(project "XMOS_demo"
 				(path "/0a855fb0-ca19-4770-811e-70d8770d7fdd/13d4ac51-413b-4f8b-9448-517b4883a5ce"
-					(reference "#PWR052")
+					(reference "#PWR053")
 					(unit 1)
 				)
@@
 		(on_board yes)
 		(dnp no)
-		(property "Reference" "C37"
+		(property "Reference" "C39"
 			(at 189.484 140.97 0)
 			(effects
@@
 			(project "XMOS_demo"
 				(path "/0a855fb0-ca19-4770-811e-70d8770d7fdd/13d4ac51-413b-4f8b-9448-517b4883a5ce"
-					(reference "C37")
+					(reference "C39")
 					(unit 1)
 				)
@@
 		(on_board yes)
 		(dnp no)
-		(property "Reference" "#PWR057"
+		(property "Reference" "#PWR058"
 			(at 187.96 156.21 0)
 			(effects
@@
 			(project "XMOS_demo"
 				(path "/0a855fb0-ca19-4770-811e-70d8770d7fdd/13d4ac51-413b-4f8b-9448-517b4883a5ce"
-					(reference "#PWR057")
+					(reference "#PWR058")
 					(unit 1)
 				)
