File: XMOS_demo/psu.kicad_sch (KiCad schematic)
At the start: 26 parts, among them U4 TLV75733PDBV, U5 TLV75718PDBV, U6 AP61200Z6

Commit message: xmos pcb work
Parts:
- TP7: footprint TestPoint:TestPoint_Keystone_5005-5009_Compact -> TestPoint:TestPoint_Pad_D2.0mm
Changed lines of the file:
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@@
 			)
 		)
-		(property "Footprint" "TestPoint:TestPoint_Keystone_5005-5009_Compact"
+		(property "Footprint" "TestPoint:TestPoint_Pad_D2.0mm"
 			(at 111.76 50.8 0)
 			(effects
